Commit message: Changes of modeling force-torque sensor in URDF

File: xarm_description/urdf/gripper/xarm_gripper.urdf.xacro (robot description, xacro)
@@ -5,8 +5,52 @@
       <joint name="${prefix}gripper_fix" type="fixed">
         <parent link="${attach_to}"/>
-        <child link="${prefix}xarm_gripper_base_link"/>
+        <child link="${prefix}ft_sensor_link"/>
         <origin xyz="${attach_xyz}" rpy="${attach_rpy}"/>
       </joint>
     </xacro:unless>
+  <!-- Modification to add Force-torque sensor model -->
+    <xacro:arg name="add_realsense_d435i" default="false"/>
+    <xacro:arg name="add_gemini2" default="false"/>
+    <xacro:property name="cam_plate_thickness" value="0.00305"/>
+    <xacro:property name="ft_length" value="0.0585"/>
+    <xacro:property name="ft_radius" value="${0.075/2.0}"/>
+    <!-- If using camera, add camera mount plate offset -->
+    <xacro:if value="${add_realsense_d435i or add_gemini2}">
+      <xacro:property name="ft_origin_z" value="${ft_length/2.0 + cam_plate_thickness}"/>
+    </xacro:if>
+    <!-- If not using camera, no camera mount plate offset -->
+    <xacro:unless value="${add_realsense_d435i or add_gemini2}">
+      <xacro:property name="ft_origin_z" value="${ft_length/2.0}"/>
+    </xacro:unless>
+    <link name="${prefix}ft_sensor_link">
+      <visual>
+        <origin xyz="0 0 ${ft_origin_z}" rpy="0 0 0"/>
+        <geometry>
+          <cylinder radius="${ft_radius}" length="${ft_length}"/>
+        </geometry>
+        <material name="Grey">
+          <color rgba="0.5 0.5 0.5 1"/>
+        </material>
+      </visual>
+      <collision>
+        <origin xyz="0 0 ${ft_origin_z}" rpy="0 0 0"/>
+        <geometry>
+          <cylinder radius="${ft_radius}" length="${ft_length}"/>
+        </geometry>
+      </collision>
+      <inertial>
+        <origin xyz="0 0 ${ft_origin_z}" rpy="0 0 0"/>
+        <mass value="0.01"/>
+        <inertia
+          ixx="1e-5" ixy="0" ixz="0"
+          iyy="1e-5" iyz="0"
+          izz="1e-5"/>
+      </inertial>
+    </link>
+    <joint name="${prefix}ft_sensor_joint" type="fixed">
+      <parent link="${prefix}ft_sensor_link"/>
+      <child link="${prefix}xarm_gripper_base_link"/>
+      <origin xyz="0 0 ${ft_length}" rpy="0 0 0"/>
+    </joint>
     <link name="${prefix}xarm_gripper_base_link">
       <inertial>

File: xarm_moveit_config/srdf/_xarm6_macro.srdf.xacro (robot description, xacro)
@@ -58,4 +58,5 @@
     <xacro:if value="${add_gripper}">
       <group name="${prefix}xarm_gripper">
+        <link name="${prefix}ft_sensor_link" />
         <link name="${prefix}xarm_gripper_base_link" />
         <link name="${prefix}left_outer_knuckle" />
@@ -92,4 +93,5 @@
       <disable_collisions link1="${prefix}left_finger" link2="${prefix}right_outer_knuckle" reason="Never" />
       <disable_collisions link1="${prefix}left_finger" link2="${prefix}xarm_gripper_base_link" reason="Never" />
+      <disable_collisions link1="${prefix}left_finger" link2="${prefix}ft_sensor_link" reason="Never" />
       <disable_collisions link1="${prefix}left_inner_knuckle" link2="${prefix}left_outer_knuckle" reason="Never" />
       <disable_collisions link1="${prefix}left_inner_knuckle" link2="${prefix}link4" reason="Never" />
@@ -100,4 +102,5 @@
       <disable_collisions link1="${prefix}left_inner_knuckle" link2="${prefix}right_outer_knuckle" reason="Never" />
       <disable_collisions link1="${prefix}left_inner_knuckle" link2="${prefix}xarm_gripper_base_link" reason="Adjacent" />
+      <disable_collisions link1="${prefix}left_inner_knuckle" link2="${prefix}ft_sensor_link" reason="Adjacent" />
       <disable_collisions link1="${prefix}left_outer_knuckle" link2="${prefix}link5" reason="Never" />
       <disable_collisions link1="${prefix}left_outer_knuckle" link2="${prefix}link6" reason="Never" />
@@ -106,4 +109,5 @@
       <disable_collisions link1="${prefix}left_outer_knuckle" link2="${prefix}right_outer_knuckle" reason="Never" />
       <disable_collisions link1="${prefix}left_outer_knuckle" link2="${prefix}xarm_gripper_base_link" reason="Adjacent" />
+      <disable_collisions link1="${prefix}left_outer_knuckle" link2="${prefix}ft_sensor_link" reason="Adjacent" />
       <disable_collisions link1="${prefix}link4" link2="${prefix}right_finger" reason="Never" />
       <disable_collisions link1="${prefix}link4" link2="${prefix}right_inner_knuckle" reason="Never" />
@@ -113,14 +117,19 @@
       <disable_collisions link1="${prefix}link5" link2="${prefix}right_outer_knuckle" reason="Never" />
       <disable_collisions link1="${prefix}link5" link2="${prefix}xarm_gripper_base_link" reason="Never" />
+      <disable_collisions link1="${prefix}link5" link2="${prefix}ft_sensor_link" reason="Never" />
       <disable_collisions link1="${prefix}link6" link2="${prefix}right_finger" reason="Never" />
       <disable_collisions link1="${prefix}link6" link2="${prefix}right_inner_knuckle" reason="Never" />
       <disable_collisions link1="${prefix}link6" link2="${prefix}right_outer_knuckle" reason="Never" />
       <disable_collisions link1="${prefix}link6" link2="${prefix}xarm_gripper_base_link" reason="Adjacent" />
+      <disable_collisions link1="${prefix}link6" link2="${prefix}ft_sensor_link" reason="Adjacent" />
       <disable_collisions link1="${prefix}right_finger" link2="${prefix}right_inner_knuckle" reason="Default" />
       <disable_collisions link1="${prefix}right_finger" link2="${prefix}right_outer_knuckle" reason="Adjacent" />
       <disable_collisions link1="${prefix}right_finger" link2="${prefix}xarm_gripper_base_link" reason="Never" />
+      <disable_collisions link1="${prefix}right_finger" link2="${prefix}ft_sensor_link" reason="Never" />
       <disable_collisions link1="${prefix}right_inner_knuckle" link2="${prefix}right_outer_knuckle" reason="Never" />
       <disable_collisions link1="${prefix}right_inner_knuckle" link2="${prefix}xarm_gripper_base_link" reason="Adjacent" />
+      <disable_collisions link1="${prefix}right_inner_knuckle" link2="${prefix}ft_sensor_link" reason="Adjacent" />
       <disable_collisions link1="${prefix}right_outer_knuckle" link2="${prefix}xarm_gripper_base_link" reason="Adjacent" />
+      <disable_collisions link1="${prefix}right_outer_knuckle" link2="${prefix}ft_sensor_link" reason="Adjacent" />
       <disable_collisions link1="${prefix}link_eef" link2="${prefix}left_finger" reason="Never" />
       <disable_collisions link1="${prefix}link_eef" link2="${prefix}left_inner_knuckle" reason="Never" />
@@ -130,4 +139,6 @@
       <disable_collisions link1="${prefix}link_eef" link2="${prefix}right_outer_knuckle" reason="Never" />
       <disable_collisions link1="${prefix}link_eef" link2="${prefix}xarm_gripper_base_link" reason="Adjacent" />
+      <disable_collisions link1="${prefix}link_eef" link2="${prefix}ft_sensor_link" reason="Adjacent" />
+      <disable_collisions link1="${prefix}xarm_gripper_base_link" link2="${prefix}ft_sensor_link" reason="Adjacent" />
     </xacro:if>
     <!-- bio gripper -->
